File: hw/console.sch (KiCad schematic (older format))
At the start: 42 parts, among them J1 Debug Port, Q4 AP2301, Q5 AP2302, Q6 AP2301, Q7 AP2302, SW2 SW_Push, SW3 SW_Push, SW4 SW_Push, SW5 SW_Push, SW6 SW_Push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

Commit message: Add missing pull down on buzzer H-bridge, 15V enable
Parts:
- added R24, R25: 100k, Resistor_SMD:R_0603_1608Metric, symbol Device:R
Connections:
- net BUZZER+: now also R24.1
- net BUZZER-: now also R25.1
- net GND: now also R24.2, R25.2
Changed lines of the file:
@@
 	1    0    0    -1
 $EndComp
-Wire Wire Line
-	9500 4450 9600 4450
 Text Notes 2100 4150 0    50   ~ 0
 Flash
@@
 Wire Wire Line
 	8200 4450 8600 4450
-Wire Wire Line
-	7800 4450 7900 4450
 $Comp
 L console:+2.8V #PWR017
@@
 Text Label 9350 1600 1    50   ~ 0
 BTN5
-Text Label 7800 4450 2    50   ~ 0
+Text Label 7600 4450 2    50   ~ 0
 BUZZER+
-Text Label 9600 4450 0    50   ~ 0
+Text Label 9800 4450 0    50   ~ 0
 BUZZER-
 Text Label 6250 3725 0    50   ~ 0
@@
 Text Notes 4700 900  2    40   ~ 0
 Active power: 0.6 mW
+$Comp
+L Device:R R24
+U 1 1 61C06CD0
+P 7600 4900
+F 0 "R24" H 7670 4946 50  0000 L CNN
+F 1 "100k" H 7670 4855 50  0000 L CNN
+F 2 "Resistor_SMD:R_0603_1608Metric" V 7530 4900 50  0001 C CNN
+F 3 "~" H 7600 4900 50  0001 C CNN
+	1    7600 4900
+	1    0    0    -1
+$EndComp
+$Comp
+L Device:R R25
+U 1 1 61C07CEC
+P 9800 4900
+F 0 "R25" H 9870 4946 50  0000 L CNN
+F 1 "100k" H 9870 4855 50  0000 L CNN
+F 2 "Resistor_SMD:R_0603_1608Metric" V 9730 4900 50  0001 C CNN
+F 3 "~" H 9800 4900 50  0001 C CNN
+	1    9800 4900
+	1    0    0    -1
+$EndComp
+Wire Wire Line
+	7600 4750 7600 4450
+Wire Wire Line
+	7600 4450 7900 4450
+Wire Wire Line
+	9500 4450 9800 4450
+Wire Wire Line
+	9800 4750 9800 4450
+$Comp
+L power:GND #PWR014
+U 1 1 61C24270
+P 7600 5350
+F 0 "#PWR014" H 7600 5100 50  0001 C CNN
+F 1 "GND" H 7605 5177 50  0001 C CNN
+F 2 "" H 7600 5350 50  0001 C CNN
+F 3 "" H 7600 5350 50  0001 C CNN
+	1    7600 5350
+	1    0    0    -1
+$EndComp
+$Comp
+L power:GND #PWR015
+U 1 1 61C283D0
+P 9800 5350
+F 0 "#PWR015" H 9800 5100 50  0001 C CNN
+F 1 "GND" H 9805 5177 50  0001 C CNN
+F 2 "" H 9800 5350 50  0001 C CNN
+F 3 "" H 9800 5350 50  0001 C CNN
+	1    9800 5350
+	1    0    0    -1
+$EndComp
+Wire Wire Line
+	9800 5050 9800 5350
+Wire Wire Line
+	7600 5050 7600 5350
 $EndSCHEMATC

Commit message: PCB improvements & enclosure
- Change revision to 2021B
- Larger battery connector holes
- Change buzzer to 8 ohm speaker
- Add enclosure CAD files
Parts:
- removed BZ1: Buzzer, console:XDCR_PS1240P02CT3, symbol Device:Buzzer
- added LS1: Speaker, console:Speaker, symbol Device:Speaker
Connections:
- net at Q4.3 (D), Q5.3 (D): now also LS1.1
- net at Q6.3 (D), Q7.3 (D): now also LS1.2
Other:
- note added: "16 ohm"
- note removed: "Active power draw: 3 mA"
Changed lines of the file:
@@
 Title "Handheld game console"
 Date "2021-11-16"
-Rev "2021A"
+Rev "2021B"
 Comp ""
 Comment1 ""
@@
 Mechanical\n
 Wire Wire Line
-	8800 4450 9200 4450
-Wire Wire Line
 	8700 5250 9200 5250
 Connection ~ 8700 5250
@@
 Text Notes 7100 3200 0    100  ~ 0
 Buzzer
-Wire Wire Line
-	8200 4450 8600 4450
 $Comp
 L console:+2.8V #PWR017
@@
 $EndComp
 $Comp
-L Device:Buzzer BZ1
-U 1 1 60DB830D
-P 8700 4350
-F 0 "BZ1" V 8549 4273 50  0000 L CNN
-F 1 "Buzzer" V 8480 4222 50  0000 L CNN
-F 2 "console:XDCR_PS1240P02CT3" V 8675 4450 50  0001 C CNN
-F 3 "~" V 8675 4450 50  0001 C CNN
-	1    8700 4350
-	0    -1   -1   0
-$EndComp
-$Comp
 L Mechanical:MountingHole H4
 U 1 1 61998BB0
@@
 	0    -1   -1   0
 $EndComp
-Text Notes 500  4275 0    40   ~ 0
-Active power draw: 3 mA
 Text Notes 3800 4500 2    40   ~ 0
 Active power: 9 mW\nStandby power: <3 uW
@@
 Wire Wire Line
 	7600 5050 7600 5350
+$Comp
+L Device:Speaker LS1
+U 1 1 61E77CF1
+P 8650 4250
+F 0 "LS1" V 8300 4275 50  0000 R CNN
+F 1 "Speaker" V 8400 4350 50  0000 R CNN
+F 2 "console:Speaker" H 8650 4050 50  0001 C CNN
+F 3 "~" H 8640 4200 50  0001 C CNN
+	1    8650 4250
+	0    -1   -1   0
+$EndComp
+Wire Wire Line
+	8750 4450 9200 4450
+Wire Wire Line
+	8200 4450 8650 4450
+Text Notes 8576 4701 0    40   ~ 0
+16 ohm
 $EndSCHEMATC
